File: atari-usb.sch (KiCad schematic (older format))
At the start: 39 parts, among them J1 USB_A, J2 DB9_Male, U1 ATmega32U4-AU, U2 TPD2EUSB30

Commit message: Revision 0 done
Parts:
- removed TP2, TP6: TestPoint, TestPoint:TestPoint_Pad_D1.0mm, symbol Connector:TestPoint
- added C9: 0.1u, Capacitor_SMD:C_0603_1608Metric, symbol Device:C
- TP1: value TestPoint -> MISO
- TP3: value TestPoint -> SCK
- TP4: value TestPoint -> MOSI
- TP5: value TestPoint -> ~RST
Connections:
- net +5V is gone; now on net VBUS: J2.7, R11.1, R12.1, R13.1, R14.1, R15.1, R3.1
- net GND: now also C9.1
- net VBUS: now also C9.2
- net at U1.10 (PB2): now also TP4.1
- net at U1.11 (PB3): now also TP1.1
- net at R3.2, U1.13 (~RESET): now also TP5.1
- net at U1.25 (PD4): now also R6.2
- net at U1.26 (PD6): now also R7.2
- net at U1.27 (PD7): now also D4.1 (K)
- net at U1.28 (PB4): now also D2.1 (K)
- net at U1.29 (PB5): now also D1.1 (K)
- net at U1.30 (PB6): now also R8.2
- net at U1.31 (PC6): now also R9.2
- net at U1.32 (PC7): now also R10.2
- net at U1.36 (PF7): now also R5.2
- net at U1.37 (PF6): now also R4.2; no longer D5.1 (K)
- net at U1.38 (PF5): no longer D4.1 (K)
- net at D3.1 (K): now also U1.8 (PB0); no longer U1.39 (PF4)
- net at U1.40 (PF1): no longer D2.1 (K)
- net at U1.41 (PF0): no longer D1.1 (K)
- net at U1.9 (PB1): now also TP3.1
- new net LED-Down: D5.1 (K), U1.39 (PF4)
- no-connect marks 0 -> 2
Other:
- moved on the sheet: D1, D2, D3, D4, D5, J2, R10, R11, R12, R13, R14, R15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

Commit message: Minor fixes during assembly
Parts:
- XTAL1: symbol dk_Crystals:NX3225GD-8MHZ-STD-CRA-3 -> atari-usb-rescue:NX3225GD-8MHZ-STD-CRA-3-dk_Crystals
Connections:
- net MOSI: now reaches TP4.1, U1.10 (PB2)
- net MISO: now reaches TP1.1, U1.11 (PB3)
- net SCK: now reaches TP3.1, U1.9 (PB1)
Changed lines of the file:
@@
 $EndComp
 $Comp
-L dk_Crystals:NX3225GD-8MHZ-STD-CRA-3 XTAL1
+L atari-usb-rescue:NX3225GD-8MHZ-STD-CRA-3-dk_Crystals XTAL1
 U 1 1 5EA6B7C6
 P 4800 2100
@@
 	6100 1500 6300 1500
 Connection ~ 6300 1500
+Text Label 6500 1950 0    50   ~ 0
+SCK
+Text Label 6500 2050 0    50   ~ 0
+MOSI
+Text Label 6500 2150 0    50   ~ 0
+MISO
 $EndSCHEMATC
